File: Pedestrian Safety.kicad_sch (KiCad schematic)
At the start: 15 parts, among them J1 Conn_01x20_Socket, J10 Conn_01x01_Pin, J2 Conn_01x20_Socket, J3 Conn_01x08_Pin, J4 Conn_01x08_Pin, J5 Conn_01x01_Pin, J6 Conn_01x01_Pin, J7 Conn_01x01_Pin, J8 Conn_01x01_Pin, J9 Conn_01x01_Pin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

Commit message: Final
Parts:
- removed J10, J5, J6, J7, J8, J9: Conn_01x01_Pin, symbol Connector:Conn_01x01_Pin
- removed J3, J4: Conn_01x08_Pin, symbol Connector:Conn_01x08_Pin
- added U2: RFM95W-915S2, RFM95W_915S2-2:XCVR_RFM95W-915S2, symbol RFM95W-915S2:RFM95W-915S2
- added U3: ~, TP4056-18650-master:TP4056-18650, symbol TP4056:TP4056
- C1: footprint (none) -> Capacitor_SMD:CP_Elec_6.3x5.7; Digikey Part Number (none) -> 732-8419-1-ND
- C2: footprint (none) -> Capacitor_SMD:C_0603_1608Metric; Digikey PN: (none) -> 1276-1013-1-ND
- J1, J2: footprint (none) -> Connector_PinHeader_2.54mm:PinHeader_1x20_P2.54mm_Vertical
- R1: footprint (none) -> Resistor_SMD:R_0603_1608Metric; Digikey PN: (none) -> P27.0KHCT-ND
- R2: footprint (none) -> Resistor_SMD:R_0603_1608Metric; Digikey PN: (none) -> 311-100KGRCT-ND
- U1: footprint Package_TO_SOT_THT:TO-92_Inline -> footprints:TO-92_MC_MCH; Digikey PN: (none) -> MCP1700-3302E/TO-ND
Connections:
- net 3V3: now also U2.13 (3.3V)
- net GND: now also U2.1 (GND), U3.2 (GND)
- net GPIO1: now also U2.2 (MISO)
- net GPIO2: now also U2.14 (DIO0)
- net GPIO38: now also U2.5 (NSS)
- net GPIO39: now also U2.4 (SCK)
- net GPIO41: now also U2.6 (RESET)
- net GPIO42: now also U2.3 (MOSI)
- net OUT+: now also U3.3 (OUT+)
